Commit message: main

File: pick_and_place/urdf/camera.urdf.xacro (robot description, xacro)
@@ -1,8 +1,8 @@
 <robot name="camera">
-    <link name="base_link"/>
+    <link name="world"/>
     <joint name="first_joint" type="fixed">
-        <parent link="base_link"/>
+        <parent link="world"/>
         <child link="camera_link"/>
-    <origin xyz="0.0 0.0 0.5" rpy="0 0.0 0.0"/>
+    <origin xyz="0.0 0.0 1.0" rpy="0.0 ${pi/4} 0.0"/>
     </joint>
     <link name="camera_link">
@@ -28,8 +28,8 @@
         </inertial>
     </link>
-    <joint name="camera_joint" type="fixed">
+    <!-- <joint name="camera_joint" type="fixed">
         <parent link="camera_link"/>
         <child link="camera_end"/>
-        <origin xyz="0.0 0.0 -0.05" rpy="0.0 0.0 0.0"/>
+        <origin xyz="0.0 0.0 0.0" rpy="0.0 0.0 0.0"/>
     </joint>
     <link name="camera_end">
@@ -39,5 +39,5 @@
             </geometry>
         </visual>
-    </link>
+    </link> -->
     <gazebo reference="camera_link">
         <material>Gazebo/Gray</material>

Commit message: main

File: pick_and_place/urdf/camera.urdf.xacro (robot description, xacro)
@@ -4,5 +4,5 @@
         <parent link="world"/>
         <child link="camera_link"/>
-    <origin xyz="0.0 0.0 1.0" rpy="0.0 ${pi/4} 0.0"/>
+    <origin xyz="0.0 0.0 1.0" rpy="0.0 ${pi/2} 0.0"/>
     </joint>
     <link name="camera_link">

Commit message: main

File: pick_and_place/urdf/camera.urdf.xacro (robot description, xacro)
@@ -1,3 +1,3 @@
-<robot name="camera">
+<robot name="camera" xmlns:xacro="http://www.ros.org/wiki/xacro">
     <link name="world"/>
     <joint name="first_joint" type="fixed">
@@ -28,16 +28,52 @@
         </inertial>
     </link>
-    <!-- <joint name="camera_joint" type="fixed">
-        <parent link="camera_link"/>
-        <child link="camera_end"/>
-        <origin xyz="0.0 0.0 0.0" rpy="0.0 0.0 0.0"/>
+    <joint name="redbox_joint" type="fixed">
+        <parent link="world"/>
+        <child link="red_box"/>
+    <origin xyz="0.0 0.0 0.0" rpy="0.0 0.0 0.0"/>
     </joint>
-    <link name="camera_end">
+    <link name="red_box">
         <visual>
+            <origin xyz="0.0 0.0 0.01" rpy="0.0 0.0 0.0"/>
             <geometry>
-                <cylinder radius="0.02" length="0.01"/>
+                <box size="0.065 0.065 0.02"/>
             </geometry>
         </visual>
-    </link> -->
+        <collision>
+            <origin xyz="0.0 0.0 0.01" rpy="0.0 0.0 0.0"/>
+            <geometry>
+                <box size="0.065 0.065 0.02"/>
+            </geometry>
+        </collision>
+        <inertial>
+            <origin xyz="0.0 0.0 0.01" rpy="0.0 0.0 0.0"/>
+            <mass value="0.200"/>
+            <inertia ixx="0.001" ixy="0.0" ixz="0.0" iyy="0.001" iyz="0.0" izz="0.001"/>
+        </inertial>
+    </link>
+    <joint name="bluebox_joint" type="fixed">
+        <parent link="world"/>
+        <child link="blue_box"/>
+    <origin xyz="0.1 0.1 0.0" rpy="0.0 0.0 0.0"/>
+    </joint>
+    <link name="blue_box">
+        <visual>
+            <origin xyz="0.0 0.0 0.01" rpy="0.0 0.0 0.0"/>
+            <geometry>
+                <box size="0.065 0.065 0.02"/>
+            </geometry>
+        </visual>
+        <collision>
+            <origin xyz="0.0 0.0 0.01" rpy="0.0 0.0 0.0"/>
+            <geometry>
+                <box size="0.065 0.065 0.02"/>
+            </geometry>
+        </collision>
+        <inertial>
+            <origin xyz="0.0 0.0 0.01" rpy="0.0 0.0 0.0"/>
+            <mass value="0.200"/>
+            <inertia ixx="0.001" ixy="0.0" ixz="0.0" iyy="0.001" iyz="0.0" izz="0.001"/>
+        </inertial>
+    </link>
     <gazebo reference="camera_link">
         <material>Gazebo/Gray</material>
@@ -77,3 +113,13 @@
         </sensor>
     </gazebo>
+    <gazebo reference="red_box">
+        <material>Gazebo/Red</material>
+        <mu1>5</mu1>
+        <mu2>5</mu2>
+    </gazebo>
+    <gazebo reference="blue_box">
+        <material>Gazebo/Blue</material>
+        <mu1>5</mu1>
+        <mu2>5</mu2>
+    </gazebo>
 </robot>

File: pick_and_place/urdf/ur3_camera.urdf.xacro (robot description, xacro)
@@ -20,7 +20,7 @@
     kinematics_file="${load_yaml('$(arg kinematics_config)')}"
   />
-  <link name="world" />
+  <link name="world_link" />
   <joint name="world_joint" type="fixed">
-    <parent link="world" />
+    <parent link="world_link" />
     <child link = "base_link" />
     <origin xyz="0.0 0.0 0.0" rpy="0.0 0.0 0.0" />

Commit message: main

File: pick_and_place/urdf/camera.urdf.xacro (robot description, xacro)
@@ -4,5 +4,5 @@
         <parent link="world"/>
         <child link="camera_link"/>
-    <origin xyz="0.0 0.0 1.0" rpy="0.0 ${pi/2} 0.0"/>
+    <origin xyz="0.0 0.0 1.0" rpy="0.0 ${pi/2} ${pi/2}"/>
     </joint>
     <link name="camera_link">
@@ -28,8 +28,32 @@
         </inertial>
     </link>
+    <joint name="bluebox_joint" type="fixed">
+        <parent link="world"/>
+        <child link="blue_box"/>
+    <origin xyz="0.0 0.0 0.0" rpy="0.0 0.0 0.0"/>
+    </joint>
+    <link name="blue_box">
+        <visual>
+            <origin xyz="0.0 0.0 0.01" rpy="0.0 0.0 0.0"/>
+            <geometry>
+                <box size="0.065 0.065 0.02"/>
+            </geometry>
+        </visual>
+        <collision>
+            <origin xyz="0.0 0.0 0.01" rpy="0.0 0.0 0.0"/>
+            <geometry>
+                <box size="0.065 0.065 0.02"/>
+            </geometry>
+        </collision>
+        <inertial>
+            <origin xyz="0.0 0.0 0.01" rpy="0.0 0.0 0.0"/>
+            <mass value="0.200"/>
+            <inertia ixx="0.001" ixy="0.0" ixz="0.0" iyy="0.001" iyz="0.0" izz="0.001"/>
+        </inertial>
+    </link>
     <joint name="redbox_joint" type="fixed">
         <parent link="world"/>
         <child link="red_box"/>
-    <origin xyz="0.0 0.0 0.0" rpy="0.0 0.0 0.0"/>
+    <origin xyz="0.1 0.1 0.0" rpy="0.0 0.0 0.0"/>
     </joint>
     <link name="red_box">
@@ -52,10 +76,10 @@
         </inertial>
     </link>
-    <joint name="bluebox_joint" type="fixed">
+    <!-- <joint name="redbox_2_joint" type="fixed">
         <parent link="world"/>
-        <child link="blue_box"/>
-    <origin xyz="0.1 0.1 0.0" rpy="0.0 0.0 0.0"/>
-    </joint>
-    <link name="blue_box">
+        <child link="red_2_box"/>
+    <origin xyz="-0.1 -0.1 0.0" rpy="0.0 0.0 ${pi/4}"/>
+    </joint> -->
+    <!-- <link name="red_2_box">
         <visual>
             <origin xyz="0.0 0.0 0.01" rpy="0.0 0.0 0.0"/>
@@ -75,5 +99,5 @@
             <inertia ixx="0.001" ixy="0.0" ixz="0.0" iyy="0.001" iyz="0.0" izz="0.001"/>
         </inertial>
-    </link>
+    </link> -->
     <gazebo reference="camera_link">
         <material>Gazebo/Gray</material>
@@ -118,4 +142,9 @@
         <mu2>5</mu2>
     </gazebo>
+    <!-- <gazebo reference="red_2_box">
+        <material>Gazebo/Red</material>
+        <mu1>5</mu1>
+        <mu2>5</mu2>
+    </gazebo> -->
     <gazebo reference="blue_box">
         <material>Gazebo/Blue</material>

Commit message: main

File: pick_and_place/urdf/camera.urdf.xacro (robot description, xacro)
@@ -1,154 +1,69 @@
-<robot name="camera" xmlns:xacro="http://www.ros.org/wiki/xacro">
-    <link name="world"/>
-    <joint name="first_joint" type="fixed">
-        <parent link="world"/>
-        <child link="camera_link"/>
-    <origin xyz="0.0 0.0 1.0" rpy="0.0 ${pi/2} ${pi/2}"/>
-    </joint>
-    <link name="camera_link">
-        <visual>
-            <origin xyz="0.0 0.0 0.0" rpy="0.0 0.0 0.0"/>
-            <geometry>
-                <box size="0.1 0.1 0.1"/>
-            </geometry>
-            <material name="Cyan">
-                <color rgba="0.0 1.0 0.0 1.0"/>
-            </material>
-        </visual>
-        <collision>
-            <origin xyz="0.0 0.0 0.0" rpy="0.0 0.0 0.0"/>
-            <geometry>
-                <box size="0.1 0.1 0.1"/>
-            </geometry>
-        </collision>
-        <inertial>
-            <origin xyz="0.0 0.0 0.0" rpy="0.0 0.0 0.0"/>
-            <mass value="0.5"/>
-            <inertia ixx="0.01" ixy="0.0" ixz="0.0" iyy="0.01" iyz="0.0" izz="0.01" />
-        </inertial>
-    </link>
-    <joint name="bluebox_joint" type="fixed">
-        <parent link="world"/>
-        <child link="blue_box"/>
-    <origin xyz="0.0 0.0 0.0" rpy="0.0 0.0 0.0"/>
-    </joint>
-    <link name="blue_box">
-        <visual>
-            <origin xyz="0.0 0.0 0.01" rpy="0.0 0.0 0.0"/>
-            <geometry>
-                <box size="0.065 0.065 0.02"/>
-            </geometry>
-        </visual>
-        <collision>
-            <origin xyz="0.0 0.0 0.01" rpy="0.0 0.0 0.0"/>
-            <geometry>
-                <box size="0.065 0.065 0.02"/>
-            </geometry>
-        </collision>
-        <inertial>
-            <origin xyz="0.0 0.0 0.01" rpy="0.0 0.0 0.0"/>
-            <mass value="0.200"/>
-            <inertia ixx="0.001" ixy="0.0" ixz="0.0" iyy="0.001" iyz="0.0" izz="0.001"/>
-        </inertial>
-    </link>
-    <joint name="redbox_joint" type="fixed">
-        <parent link="world"/>
-        <child link="red_box"/>
-    <origin xyz="0.1 0.1 0.0" rpy="0.0 0.0 0.0"/>
-    </joint>
-    <link name="red_box">
-        <visual>
-            <origin xyz="0.0 0.0 0.01" rpy="0.0 0.0 0.0"/>
-            <geometry>
-                <box size="0.065 0.065 0.02"/>
-            </geometry>
-        </visual>
-        <collision>
-            <origin xyz="0.0 0.0 0.01" rpy="0.0 0.0 0.0"/>
-            <geometry>
-                <box size="0.065 0.065 0.02"/>
-            </geometry>
-        </collision>
-        <inertial>
-            <origin xyz="0.0 0.0 0.01" rpy="0.0 0.0 0.0"/>
-            <mass value="0.200"/>
-            <inertia ixx="0.001" ixy="0.0" ixz="0.0" iyy="0.001" iyz="0.0" izz="0.001"/>
-        </inertial>
-    </link>
-    <!-- <joint name="redbox_2_joint" type="fixed">
-        <parent link="world"/>
-        <child link="red_2_box"/>
-    <origin xyz="-0.1 -0.1 0.0" rpy="0.0 0.0 ${pi/4}"/>
-    </joint> -->
-    <!-- <link name="red_2_box">
-        <visual>
-            <origin xyz="0.0 0.0 0.01" rpy="0.0 0.0 0.0"/>
-            <geometry>
-                <box size="0.065 0.065 0.02"/>
-            </geometry>
-        </visual>
-        <collision>
-            <origin xyz="0.0 0.0 0.01" rpy="0.0 0.0 0.0"/>
-            <geometry>
-                <box size="0.065 0.065 0.02"/>
-            </geometry>
-        </collision>
-        <inertial>
-            <origin xyz="0.0 0.0 0.01" rpy="0.0 0.0 0.0"/>
-            <mass value="0.200"/>
-            <inertia ixx="0.001" ixy="0.0" ixz="0.0" iyy="0.001" iyz="0.0" izz="0.001"/>
-        </inertial>
-    </link> -->
-    <gazebo reference="camera_link">
-        <material>Gazebo/Gray</material>
-        <sensor type="camera" name="camera1">
-            <update_rate>30.0</update_rate>
-            <camera name="head">
-                <horizontal_fov>1.3962634</horizontal_fov>
-                <image>
-                <width>640</width>
-                <height>360</height>
-                <format>R8G8B8</format>
-                </image>
-                <clip>
-                <near>0.02</near>
-                <far>300</far>
-                </clip>
-                <noise>
-                <type>gaussian</type>
-                <mean>0.0</mean>
-                <stddev>0.007</stddev>
-                </noise>
-            </camera>
-            <plugin name="camera_controller" filename="libgazebo_ros_camera.so">
-                <alwaysOn>true</alwaysOn>
-                <updateRate>0.0</updateRate>
-                <cameraName>camera</cameraName>
-                <imageTopicName>image_raw</imageTopicName>
-                <cameraInfoTopicName>camera_info</cameraInfoTopicName>
-                <frameName>camera_link</frameName>
-                <hackBaseline>0.07</hackBaseline>
-                <distortionK1>0.0</distortionK1>
-                <distortionK2>0.0</distortionK2>
-                <distortionK3>0.0</distortionK3>
-                <distortionT1>0.0</distortionT1>
-                <distortionT2>0.0</distortionT2>
-            </plugin>
-        </sensor>
-    </gazebo>
-    <gazebo reference="red_box">
-        <material>Gazebo/Red</material>
-        <mu1>5</mu1>
-        <mu2>5</mu2>
-    </gazebo>
-    <!-- <gazebo reference="red_2_box">
-        <material>Gazebo/Red</material>
-        <mu1>5</mu1>
-        <mu2>5</mu2>
-    </gazebo> -->
-    <gazebo reference="blue_box">
-        <material>Gazebo/Blue</material>
-        <mu1>5</mu1>
-        <mu2>5</mu2>
-    </gazebo>
+<?xml version="1.0"?>
+<robot xmlns:xacro="http://www.ros.org/wiki/xacro">
+    <xacro:macro name="camera" params="parent *joint_origin">
+        <joint name="$camera_joint" type="fixed">
+            <xacro:insert_block name="joint_origin"/>
+            <parent link="${parent}"/>
+            <child link="camera_link"/>
+        </joint>
+        <link name="camera_link">
+            <visual>
+                <origin xyz="0.0 0.0 0.0" rpy="0.0 0.0 0.0"/>
+                <geometry>
+                    <box size="0.1 0.1 0.1"/>
+                </geometry>
+                <material name="Cyan">
+                    <color rgba="0.0 1.0 0.0 1.0"/>
+                </material>
+            </visual>
+            <collision>
+                <origin xyz="0.0 0.0 0.0" rpy="0.0 0.0 0.0"/>
+                <geometry>
+                    <box size="0.1 0.1 0.1"/>
+                </geometry>
+            </collision>
+            <inertial>
+                <origin xyz="0.0 0.0 0.0" rpy="0.0 0.0 0.0"/>
+                <mass value="0.5"/>
+                <inertia ixx="0.01" ixy="0.0" ixz="0.0" iyy="0.01" iyz="0.0" izz="0.01" />
+                </inertial>
+        </link>
+        <gazebo reference="camera_link">
+            <material>Gazebo/Gray</material>
+            <sensor type="camera" name="camera1">
+                <update_rate>30.0</update_rate>
+                <camera name="head">
+                    <horizontal_fov>1.3962634</horizontal_fov>
+                    <image>
+                    <width>640</width>
+                    <height>360</height>
+                    <format>R8G8B8</format>
+                    </image>
+                    <clip>
+                    <near>0.02</near>
+                    <far>300</far>
+                    </clip>
+                    <noise>
+                    <type>gaussian</type>
+                    <mean>0.0</mean>
+                    <stddev>0.007</stddev>
+                    </noise>
+                </camera>
+                <plugin name="camera_controller" filename="libgazebo_ros_camera.so">
+                    <alwaysOn>true</alwaysOn>
+                    <updateRate>0.0</updateRate>
+                    <cameraName>camera</cameraName>
+                    <imageTopicName>image_raw</imageTopicName>
+                    <cameraInfoTopicName>camera_info</cameraInfoTopicName>
+                    <frameName>camera_link</frameName>
+                    <hackBaseline>0.07</hackBaseline>
+                    <distortionK1>0.0</distortionK1>
+                    <distortionK2>0.0</distortionK2>
+                    <distortionK3>0.0</distortionK3>
+                    <distortionT1>0.0</distortionT1>
+                    <distortionT2>0.0</distortionT2>
+                </plugin>
+            </sensor>
+        </gazebo>
+    </xacro:macro>
 </robot>

File: pick_and_place/urdf/redbox.urdf.xacro (robot description, xacro)
@@ -1,30 +1,39 @@
 <?xml version="1.0"?>
-<robot name="red_box">
-<link name="base_link">
-  <collision>
-    <origin xyz="0 0 0.02" rpy="0 0 0"/>
-    <geometry>
-      <box size="0.1 0.075 0.025" />
-    </geometry>
-  </collision>
-  <visual>
-    <origin xyz="0 0 0.02" rpy="0 0 0"/>
-    <geometry>
-      <box size="0.1 0.075 0.025" />
-    </geometry>
-  </visual>
-  <inertial>
-    <origin xyz="0 0 0.02" rpy="0 0 0" />
-    <mass value="0.05" />
-    <inertia
-      ixx="0.001" ixy="0.0"  ixz="0.0"
-      iyy="0.001" iyz="0.0"
-      izz="0.001" />
-  </inertial>
-  </link>
-<gazebo reference="base_link">
-  <material>Gazebo/Red</material>
-    <mu1>5</mu1>
-    <mu2>5</mu2>
-</gazebo>
+<robot xmlns:xacro="http://www.ros.org/wiki/xacro">
+  <xacro:macro name="red_box" params="parent *joint_origin">
+  <material name="red">
+    <color rgba="1.0 0.0 0.0 1.0"/>
+  </material>
+    <joint name="red_box_joint" type="revolute">
+      <xacro:insert_block name="joint_origin"/>
+      <parent link="${parent}"/>
+      <child link="red_box"/>
+    </joint>
+    <link name="red_box">
+      <visual>
+        <origin xyz="0.0 0.0 0.01" rpy="0.0 0.0 0.0"/>
+        <geometry>
+          <box size="0.065 0.065 0.02"/>
+        </geometry>
+        <material name="red">
+        </material>
+      </visual>
+      <collision>
+        <origin xyz="0.0 0.0 0.01" rpy="0.0 0.0 0.0"/>
+        <geometry>
+          <box size="0.065 0.065 0.02"/>
+        </geometry>
+      </collision>
+      <inertial>
+        <origin xyz="0.0 0.0 0.01" rpy="0.0 0.0 0.0"/>
+        <mass value="0.200"/>
+        <inertia ixx="0.001" ixy="0.0" ixz="0.0" iyy="0.001" iyz="0.0" izz="0.001"/>
+      </inertial>
+    </link>
+    <gazebo reference="red_box">
+        <material>Gazebo/Red</material>
+        <mu1>5</mu1>
+        <mu2>5</mu2>
+    </gazebo>
+  </xacro:macro>
 </robot>

File: pick_and_place/urdf/ur3_camera.urdf.xacro (robot description, xacro)
@@ -3,5 +3,4 @@
        name="ur3" >
   <xacro:arg name="transmission_hw_interface" default="hardware_interface/PositionJointInterface"/>
-  <xacro:property name="camera_link" value="0.02" /> <!-- Size of square 'camera' box -->
   <!-- common stuff -->
   <xacro:include filename="$(find ur_description)/urdf/common.gazebo.xacro" />
@@ -20,79 +19,21 @@
     kinematics_file="${load_yaml('$(arg kinematics_config)')}"
   />
-  <link name="world_link" />
-  <joint name="world_joint" type="fixed">
-    <parent link="world_link" />
-    <child link = "base_link" />
-    <origin xyz="0.0 0.0 0.0" rpy="0.0 0.0 0.0" />
+  <link name="world_link"/>
+  <joint name="ur_base_joint" type="fixed">
+    <origin xyz="0.0 0.0 0.25" rpy="0.0 0.0 0.0"/>
+    <parent link="pedestal_link"/>
+    <child link="base_link"/>
   </joint>
-  <joint name="camera_joint" type="fixed">
-    <axis xyz="0 0 0" />
-    <origin xyz="0 0 0.04" rpy="0 0 ${pi/2}"/>
-    <parent link="wrist_2_link"/>
-    <child link="camera_link"/>
-  </joint>
-  <!-- Camera -->
-  <link name="camera_link">
-    <collision>
-      <origin xyz="0 0 0" rpy="0 0 0"/>
-      <geometry>
-    <box size="${camera_link} ${camera_link} ${camera_link}"/>
-      </geometry>
-    </collision>
-    <visual>
-      <origin xyz="0 0 0" rpy="0 0 0"/>
-      <geometry>
-    <box size="${camera_link} ${camera_link} ${camera_link}"/>
-      </geometry>
-      <material name="red">
-        <color rgba="1.0 0.0 0.0 2.0"/>
-      </material>
-    </visual>
-    <inertial>
-      <mass value="1e-5" />
-      <origin xyz="0 0 0" rpy="0 0 0"/>
-      <inertia ixx="1e-6" ixy="0" ixz="0" iyy="1e-6" iyz="0" izz="1e-6" />
-    </inertial>
-  </link>
-  <!-- camera -->
-  <gazebo reference="camera_link">
-    <material>Gazebo/Red</material>
-    <sensor type="camera" name="camera1">
-      <update_rate>30.0</update_rate>
-      <camera name="head">
-        <horizontal_fov>1.3962634</horizontal_fov>
-        <image>
-          <width>800</width>
-          <height>800</height>
-          <format>R8G8B8</format>
-        </image>
-        <clip>
-          <near>0.02</near>
-          <far>300</far>
-        </clip>
-        <noise>
-          <type>gaussian</type>
-          <!-- Noise is sampled independently per pixel on each frame.
-               That pixel's noise value is added to each of its color
-               channels, which at that point lie in the range [0,1]. -->
-          <mean>0.0</mean>
-          <stddev>0.007</stddev>
-        </noise>
-      </camera>
-      <plugin name="camera_controller" filename="libgazebo_ros_camera.so">
-        <alwaysOn>true</alwaysOn>
-        <updateRate>0.0</updateRate>
-        <cameraName>ur3/camera1</cameraName>
-        <imageTopicName>image_raw</imageTopicName>
-        <cameraInfoTopicName>camera_info</cameraInfoTopicName>
-        <frameName>camera_link</frameName>
-        <hackBaseline>0.07</hackBaseline>
-        <distortionK1>0.0</distortionK1>
-        <distortionK2>0.0</distortionK2>
-        <distortionK3>0.0</distortionK3>
-        <distortionT1>0.0</distortionT1>
-        <distortionT2>0.0</distortionT2>
-      </plugin>
-    </sensor>
-  </gazebo>
-</robot>
+  <xacro:include filename="$(find pick_and_place)/urdf/redbox.urdf.xacro"/>
+  <xacro:include filename="$(find pick_and_place)/urdf/camera.urdf.xacro"/>
+  <xacro:include filename="$(find pick_and_place)/urdf/pedestal.urdf.xacro"/>
+  <xacro:red_box parent="world_link">
+    <origin xyz="1.0 1.0 0.0"/>
+  </xacro:red_box>
+  <xacro:camera parent="world_link">
+    <origin xyz="0.0 0.0 2.0" rpy="0.0 ${pi/2} ${pi/2}"/>
+  </xacro:camera>
+  <xacro:pedestal parent="world_link">
+    <origin xyz="0.0 0.0 0.25"/>
+  </xacro:pedestal>
+  </robot>
