Commit message: main

File: pick_and_place/urdf/bin.urdf.xacro (robot description, xacro)
@@ -1,35 +1,35 @@
 <?xml version="1.0"?>
 <robot xmlns:xacro="http://www.ros.org/wiki/xacro">
-    <xacro:macro name="pedestal" params="parent *joint_origin">
-        <material name="green">
-            <color rgba="0.0 1.0 0.0 1.0"/>
+    <xacro:macro name="bin" params="parent *joint_origin">
+        <material name="blue">
+            <color rgba="0.0 0.0 1.0 1.0"/>
         </material>
-        <joint name="pedestal_joint" type="fixed">
+        <joint name="bin_joint" type="fixed">
             <xacro:insert_block name="joint_origin"/>
             <parent link="${parent}"/>
-            <child link="pedestal_link"/>
+            <child link="bin_link"/>
         </joint>
-        <link name="pedestal_link">
+        <link name="bin_link">
             <inertial>
                 <origin xyz="0.0 0.0 0.0" rpy="0.0 0.0 0.0"/>
-                <mass value="44.391"/>
-                <inertia ixx="3.739" ixy="0.0" ixz="1.393e-10" iyy="3.739" iyz="0.0" izz="0.08"/>
+                <mass value="6.614"/>
+                <inertia ixx="0.098" ixy="0.0" ixz="0.0" iyy="0.098" iyz="0.0" izz="0.123"/>
             </inertial>
             <visual>
                 <origin xyz="0.0 0.0 0.0" rpy="0.0 0.0 0.0"/>
                 <geometry>
-                    <cylinder radius="0.06" length="0.5"/>
+                    <mesh filename="package://pick_and_place/stl/bin.stl"/>
                 </geometry>
-                <material name="green"/>
+                <material name="blue"/>
             </visual>
             <collision>
                 <origin xyz="0.0 0.0 0.0" rpy="0.0 0.0 0.0"/>
                 <geometry>
-                    <cylinder radius="0.06" length="0.5"/>
+                    <mesh filename="package://pick_and_place/stl/bin.stl"/>
                 </geometry>
             </collision>
         </link>
-        <gazebo reference="pedestal_link">
-            <material>Gazebo/Green</material>
+        <gazebo reference="bin_link">
+            <material>Gazebo/Blue</material>
         </gazebo>
     </xacro:macro>

File: pick_and_place/urdf/desk.urdf.xacro (robot description, xacro)
@@ -2,4 +2,7 @@
 <robot xmlns:xacro="http://www.ros.org/wiki/xacro">
     <xacro:macro name="desk" params="parent *joint_origin">
+        <material name="green">
+            <color rgba="0.0 1.0 0.0 1.0"/>
+        </material>
         <joint name="desk_joint" type="fixed">
             <xacro:insert_block name="joint_origin"/>
@@ -10,6 +13,6 @@
             <inertial>
                 <origin xyz="0.0 0.0 0.0" rpy="0.0 0.0 0.0"/>
-                <mass value="0.0"/>
-                <inertia ixx="0.0" ixy="0.0" ixz="0.0" iyy="0.0" iyz="0.0" izz="0.0"/>
+                <mass value="14.44"/>
+                <inertia ixx="1.801" ixy="0.0" ixz="0.0" iyy="1.801" iyz="0.0" izz="0.465"/>
             </inertial>
             <visual>
@@ -18,4 +21,5 @@
                     <mesh filename="package://pick_and_place/stl/desk.stl"/>
                 </geometry>
+                <material name="green"/>
             </visual>
             <collision>
@@ -26,4 +30,7 @@
             </collision>
         </link>
+        <gazebo reference="desk_link">
+            <material>Gazebo/Green</material>
+        </gazebo>
     </xacro:macro>
 </robot>

File: pick_and_place/urdf/ur3_camera.urdf.xacro (robot description, xacro)
@@ -29,4 +29,5 @@
   <xacro:include filename="$(find pick_and_place)/urdf/pedestal.urdf.xacro"/>
   <xacro:include filename="$(find pick_and_place)/urdf/desk.urdf.xacro"/>
+  <xacro:include filename="$(find pick_and_place)/urdf/bin.urdf.xacro"/>
   <xacro:red_box parent="desk_link">
     <origin xyz="0.1 0.1 0.4"/>
@@ -41,3 +42,6 @@
     <origin xyz="0.3 0.0 0.0"/>
   </xacro:desk>
+  <xacro:bin parent="world_link">
+    <origin xyz="0.0 0.6 0.0"/>
+  </xacro:bin>
   </robot>

Commit message: main

File: pick_and_place/urdf/bin.urdf.xacro (robot description, xacro)
@@ -19,5 +19,5 @@
                 <origin xyz="0.0 0.0 0.0" rpy="0.0 0.0 0.0"/>
                 <geometry>
-                    <mesh filename="package://pick_and_place/stl/bin.stl"/>
+                    <mesh filename="package://pick_and_place/dae/bin.dae"/>
                 </geometry>
                 <material name="blue"/>
@@ -26,5 +26,5 @@
                 <origin xyz="0.0 0.0 0.0" rpy="0.0 0.0 0.0"/>
                 <geometry>
-                    <mesh filename="package://pick_and_place/stl/bin.stl"/>
+                    <mesh filename="package://pick_and_place/dae/bin.dae"/>
                 </geometry>
             </collision>

File: pick_and_place/urdf/desk.urdf.xacro (robot description, xacro)
@@ -19,5 +19,5 @@
                 <origin xyz="0.0 0.0 0.0" rpy="0.0 0.0 0.0"/>
                 <geometry>
-                    <mesh filename="package://pick_and_place/stl/desk.stl"/>
+                    <mesh filename="package://pick_and_place/dae/table.dae"/>
                 </geometry>
                 <material name="green"/>
@@ -26,5 +26,5 @@
                 <origin xyz="0.0 0.0 0.0" rpy="0.0 0.0 0.0"/>
                 <geometry>
-                    <mesh filename="package://pick_and_place/stl/desk.stl"/>
+                    <mesh filename="package://pick_and_place/dae/table.dae"/>
                 </geometry>
             </collision>
