Commit message: main

File: pick_and_place/urdf/camera_v2.urdf.xacro (robot description, xacro)
@@ -3,5 +3,4 @@
         <link name="world_link"/>
         <joint name="camera_joint" type="fixed">
-            <origin xyz="0.2 0.0 2.0" rpy="0.0 ${pi/2} ${pi/2}"/>
             <parent link="world_link"/>
             <child link="camera_link"/>
@@ -9,5 +8,6 @@
         <link name="camera_link">
             <visual>
-                <origin xyz="0.0 0.0 0.0" rpy="0.0 0.0 0.0"/>
+                <!-- <origin xyz="0.0 0.0 0.0" rpy="0.0 0.0 0.0"/> -->
+                <origin xyz="0.0 0.0 0.0" rpy="0.0 ${pi/2} ${pi/2}"/>
                 <geometry>
                     <box size="0.1 0.1 0.1"/>
@@ -18,5 +18,6 @@
             </visual>
             <collision>
-                <origin xyz="0.0 0.0 0.0" rpy="0.0 0.0 0.0"/>
+                <!-- <origin xyz="0.0 0.0 0.0" rpy="0.0 0.0 0.0"/> -->
+                <origin xyz="0.0 0.0 0.0" rpy="0.0 ${pi/2} ${pi/2}"/>
                 <geometry>
                     <box size="0.1 0.1 0.1"/>
@@ -24,5 +25,6 @@
             </collision>
             <inertial>
-                <origin xyz="0.0 0.0 0.0" rpy="0.0 0.0 0.0"/>
+                <!-- <origin xyz="0.0 0.0 0.0" rpy="0.0 0.0 0.0"/> -->
+                <origin xyz="0.0 0.0 0.0" rpy="0.0 ${pi/2} ${pi/2}"/>
                 <mass value="0.5"/>
                 <inertia ixx="0.01" ixy="0.0" ixz="0.0" iyy="0.01" iyz="0.0" izz="0.01" />

File: pick_and_place/urdf/ur3_camera.urdf.xacro (robot description, xacro)
@@ -54,5 +54,5 @@
     <parent link="world_link"/>
     <child link="camera_link"/>
-</joint>
+  </joint>
 <link name="camera_link">
   <visual>
