Commit message: main

File: pick_and_place/urdf/bin_v2.urdf.xacro (robot description, xacro)
@@ -1,11 +1,10 @@
 <?xml version="1.0"?>
-<robot xmlns:xacro="http://www.ros.org/wiki/xacro">
-    <xacro:macro name="bin" params="parent *joint_origin">
+<robot name='bin'>
         <material name="blue">
             <color rgba="0.0 0.0 1.0 1.0"/>
         </material>
+        <link name="world_link"/>
         <joint name="bin_joint" type="fixed">
-            <xacro:insert_block name="joint_origin"/>
-            <parent link="${parent}"/>
+            <parent link="world_link"/>
             <child link="bin_link"/>
         </joint>
@@ -35,4 +34,3 @@
             <material>Gazebo/Blue</material>
         </gazebo>
-    </xacro:macro>
 </robot>

File: pick_and_place/urdf/camera_v2.urdf.xacro (robot description, xacro)
@@ -1,8 +1,8 @@
 <?xml version="1.0"?>
-<robot xmlns:xacro="http://www.ros.org/wiki/xacro">
-    <xacro:macro name="camera" params="parent *joint_origin">
-        <joint name="$camera_joint" type="fixed">
-            <xacro:insert_block name="joint_origin"/>
-            <parent link="${parent}"/>
+<robot name='camera'>
+        <link name="world_link"/>
+        <joint name="camera_joint" type="fixed">
+            <origin xyz="0.2 0.0 2.0" rpy="0.0 ${pi/2} ${pi/2}"/>
+            <parent link="world_link"/>
             <child link="camera_link"/>
         </joint>
@@ -66,4 +66,3 @@
             </sensor>
         </gazebo>
-    </xacro:macro>
 </robot>

File: pick_and_place/urdf/desk_v2.urdf.xacro (robot description, xacro)
@@ -1,11 +1,10 @@
 <?xml version="1.0"?>
-<robot xmlns:xacro="http://www.ros.org/wiki/xacro">
-    <xacro:macro name="desk" params="parent *joint_origin">
+<robot name='desk'>
         <material name="green">
             <color rgba="0.0 1.0 0.0 1.0"/>
         </material>
+        <link name="world_link"/>
         <joint name="desk_joint" type="fixed">
-            <xacro:insert_block name="joint_origin"/>
-            <parent link="${parent}"/>
+            <parent link="world_link"/>
             <child link="desk_link"/>
         </joint>
@@ -35,4 +34,3 @@
             <material>Gazebo/Green</material>
         </gazebo>
-    </xacro:macro>
 </robot>

File: pick_and_place/urdf/ur3_camera.urdf.xacro (robot description, xacro)
@@ -20,28 +20,100 @@
   />
   <link name="world_link"/>
-  <joint name="ur_base_joint" type="fixed">
-    <origin xyz="0.0 0.0 0.25" rpy="0.0 0.0 0.0"/>
+  <link name="pedestal_link">
+    <inertial>
+        <origin xyz="0.0 0.0 0.0" rpy="0.0 0.0 0.0"/>
+        <mass value="44.391"/>
+        <inertia ixx="3.739" ixy="0.0" ixz="1.393e-10" iyy="3.739" iyz="0.0" izz="0.08"/>
+    </inertial>
+    <visual>
+        <origin xyz="0.0 0.0 0.0" rpy="0.0 0.0 0.0"/>
+        <geometry>
+            <cylinder radius="0.06" length="0.5"/>
+        </geometry>
+        <material name="green"/>
+    </visual>
+    <collision>
+        <origin xyz="0.0 0.0 0.0" rpy="0.0 0.0 0.0"/>
+        <geometry>
+            <cylinder radius="0.06" length="0.5"/>
+        </geometry>
+    </collision>
+  </link>
+  <joint name="world_joint" type="fixed">
+    <origin xyz="0.0 0.0 0.25"/>
+    <parent link="world_link"/>
+    <child link="pedestal_link"/>
+  </joint>
+  <joint name="pedestal_joint" type="fixed">
+    <origin xyz="0.0 0.0 0.25"/>
     <parent link="pedestal_link"/>
     <child link="base_link"/>
   </joint>
-  <xacro:include filename="$(find pick_and_place)/urdf/redbox.urdf.xacro"/>
-  <xacro:include filename="$(find pick_and_place)/urdf/camera.urdf.xacro"/>
-  <xacro:include filename="$(find pick_and_place)/urdf/pedestal.urdf.xacro"/>
-  <xacro:include filename="$(find pick_and_place)/urdf/desk.urdf.xacro"/>
-  <xacro:include filename="$(find pick_and_place)/urdf/bin.urdf.xacro"/>
-  <xacro:red_box parent="desk_link">
-    <origin xyz="0.1 0.1 0.4"/>
-  </xacro:red_box>
-  <xacro:camera parent="world_link">
-    <origin xyz="0.2 0.0 2.0" rpy="0.0 ${pi/2} ${pi/2}"/>
-  </xacro:camera>
-  <xacro:pedestal parent="world_link">
-    <origin xyz="0.0 0.0 0.25"/>
-  </xacro:pedestal>
-  <xacro:desk parent="world_link">
-    <origin xyz="0.3 0.0 0.0"/>
-  </xacro:desk>
-  <xacro:bin parent="world_link">
-    <origin xyz="0.0 0.6 0.0"/>
-  </xacro:bin>
-  </robot>
+  <joint name="camera_joint" type="fixed">
+    <origin xyz="0.0 0.0 2.0" rpy="0.0 ${pi/2} ${pi/2}"/>
+    <parent link="world_link"/>
+    <child link="camera_link"/>
+</joint>
+<link name="camera_link">
+  <visual>
+    <origin xyz="0.0 0.0 0.0" rpy="0.0 0.0 0.0"/>
+    <geometry>
+      <box size="0.1 0.1 0.1"/>
+    </geometry>
+    <material name="Cyan">
+      <color rgba="0.0 1.0 0.0 1.0"/>
+    </material>
+  </visual>
+  <collision>
+    <origin xyz="0.0 0.0 0.0" rpy="0.0 0.0 0.0"/>
+    <geometry>
+      <box size="0.1 0.1 0.1"/>
+    </geometry>
+  </collision>
+  <inertial>
+    <origin xyz="0.0 0.0 0.0" rpy="0.0 0.0 0.0"/>
+    <mass value="0.5"/>
+    <inertia ixx="0.01" ixy="0.0" ixz="0.0" iyy="0.01" iyz="0.0" izz="0.01" />
+  </inertial>
+</link>
+<gazebo reference="pedestal_link">
+  <material>Gazebo/Green</material>
+</gazebo>
+<gazebo reference="camera_link">
+  <material>Gazebo/Gray</material>
+  <sensor type="camera" name="camera1">
+      <update_rate>30.0</update_rate>
+      <camera name="head">
+          <horizontal_fov>1.3962634</horizontal_fov>
+          <image>
+          <width>640</width>
+          <height>360</height>
+          <format>R8G8B8</format>
+          </image>
+          <clip>
+          <near>0.02</near>
+          <far>300</far>
+          </clip>
+          <noise>
+          <type>gaussian</type>
+          <mean>0.0</mean>
+          <stddev>0.007</stddev>
+          </noise>
+      </camera>
+      <plugin name="camera_controller" filename="libgazebo_ros_camera.so">
+          <alwaysOn>true</alwaysOn>
+          <updateRate>0.0</updateRate>
+          <cameraName>camera</cameraName>
+          <imageTopicName>image_raw</imageTopicName>
+          <cameraInfoTopicName>camera_info</cameraInfoTopicName>
+          <frameName>camera_link</frameName>
+          <hackBaseline>0.07</hackBaseline>
+          <distortionK1>0.0</distortionK1>
+          <distortionK2>0.0</distortionK2>
+          <distortionK3>0.0</distortionK3>
+          <distortionT1>0.0</distortionT1>
+          <distortionT2>0.0</distortionT2>
+      </plugin>
+  </sensor>
+</gazebo>
+</robot>

Commit message: main

File: pick_and_place/urdf/bin_v2.urdf.xacro (robot description, xacro)
@@ -4,7 +4,7 @@
             <color rgba="0.0 0.0 1.0 1.0"/>
         </material>
-        <link name="world_link"/>
+        <link name="world"/>
         <joint name="bin_joint" type="fixed">
-            <parent link="world_link"/>
+            <parent link="world"/>
             <child link="bin_link"/>
         </joint>

File: pick_and_place/urdf/camera_v2.urdf.xacro (robot description, xacro)
@@ -1,7 +1,7 @@
 <?xml version="1.0"?>
 <robot name='camera'>
-        <link name="world_link"/>
+        <link name="world"/>
         <joint name="camera_joint" type="fixed">
-            <parent link="world_link"/>
+            <parent link="world"/>
             <child link="camera_link"/>
         </joint>

File: pick_and_place/urdf/desk_v2.urdf.xacro (robot description, xacro)
@@ -4,7 +4,7 @@
             <color rgba="0.0 1.0 0.0 1.0"/>
         </material>
-        <link name="world_link"/>
+        <link name="world"/>
         <joint name="desk_joint" type="fixed">
-            <parent link="world_link"/>
+            <parent link="world"/>
             <child link="desk_link"/>
         </joint>

File: pick_and_place/urdf/redbox_v2.urdf.xacro (robot description, xacro)
@@ -4,7 +4,7 @@
     <color rgba="1.0 0.0 0.0 1.0"/>
   </material>
-    <link name="world_link"/>
+    <link name="world"/>
     <joint name="red_box_joint" type="fixed">
-      <parent link="world_link"/>
+      <parent link="world"/>
       <child link="red_box"/>
     </joint>

File: pick_and_place/urdf/ur3_camera.urdf.xacro (robot description, xacro)
@@ -1,81 +1,119 @@
 <?xml version="1.0"?>
-<robot xmlns:xacro="http://www.ros.org/wiki/xacro" name="ur3e_gripper">
-  <!--xacro:include filename="$(find ur5_description)/urdf/ur5_joint_limited_robot.urdf.xacro" /-->
-  <xacro:include filename="$(find ur_e_description)/urdf/ur3e_joint_limited_robot.urdf.xacro" />
-  <xacro:include filename="$(find ur_e_description)/urdf/hande_camera.urdf.xacro" />
-  <!-- Robotiq Coupler -->
-  <!--  + Height added by the coupler: 8mm -->
-  <!--  + Reference frame: at the middle (4mm) -->
-  <link name="robotiq_coupler">
+<robot xmlns:xacro="http://wiki.ros.org/xacro"
+       name="ur3" >
+  <xacro:arg name="transmission_hw_interface" default="hardware_interface/PositionJointInterface"/>
+  <!-- common stuff -->
+  <xacro:include filename="$(find ur_description)/urdf/common.gazebo.xacro" />
+  <!-- ur3 -->
+  <xacro:include filename="$(find ur_description)/urdf/ur3.urdf.xacro" />
+  <!-- arm -->
+  <xacro:arg name="kinematics_config" default="$(find ur_description)/config/ur3_default.yaml"/>
+  <xacro:ur3_robot prefix="" joint_limited="true"
+    shoulder_pan_lower_limit="${-pi}" shoulder_pan_upper_limit="${pi}"
+    shoulder_lift_lower_limit="${-pi}" shoulder_lift_upper_limit="${pi}"
+    elbow_joint_lower_limit="${-pi}" elbow_joint_upper_limit="${pi}"
+    wrist_1_lower_limit="${-pi}" wrist_1_upper_limit="${pi}"
+    wrist_2_lower_limit="${-pi}" wrist_2_upper_limit="${pi}"
+    wrist_3_lower_limit="${-pi}" wrist_3_upper_limit="${pi}"
+    transmission_hw_interface="$(arg transmission_hw_interface)"
+    kinematics_file="${load_yaml('$(arg kinematics_config)')}"
+  />
+  <link name="world"/>
+  <link name="pedestal_link">
+    <inertial>
+        <origin xyz="0.0 0.0 0.0" rpy="0.0 0.0 0.0"/>
+        <mass value="44.391"/>
+        <inertia ixx="3.739" ixy="0.0" ixz="1.393e-10" iyy="3.739" iyz="0.0" izz="0.08"/>
+    </inertial>
     <visual>
-      <geometry>
-        <mesh filename="package://arm_and_gripper/meshes/robotiq_85_coupler.stl" />
-      </geometry>
-      <material name="flat_black"/>
+        <origin xyz="0.0 0.0 0.0" rpy="0.0 0.0 0.0"/>
+        <geometry>
+            <cylinder radius="0.06" length="0.5"/>
+        </geometry>
+        <material name="green"/>
     </visual>
     <collision>
-      <geometry>
-        <mesh filename="package://arm_and_gripper/meshes/robotiq_85_coupler.stl" />
-      </geometry>
+        <origin xyz="0.0 0.0 0.0" rpy="0.0 0.0 0.0"/>
+        <geometry>
+            <cylinder radius="0.06" length="0.5"/>
+        </geometry>
     </collision>
-    <inertial>
-      <!--origin xyz="2.073e-05   1.45286e-03  -1.1049e-03" rpy="0 0 0" /-->
-      <mass value="0.168" />
-      <inertia ixx="6.69695624e-05" ixy="5.21511788e-09" ixz="-2.74383009e-08"
-               iyy="7.85088161e-05" iyz="5.41105193e-07" izz="1.41819717e-04"/>
-    </inertial>
   </link>
-  <joint name="robotiq_coupler_joint" type="fixed">
-    <!--origin xyz="0 0 0.004" rpy="0 0 ${pi}" /-->
-    <parent link="tool0"/>
-    <child link="robotiq_coupler"/>
+  <joint name="world_joint" type="fixed">
+    <origin xyz="0.0 0.0 0.25"/>
+    <parent link="world"/>
+    <child link="pedestal_link"/>
   </joint>
-  <gazebo reference="robotiq_coupler">
-    <mu1>0.9</mu1>
-    <mu2>0.9</mu2>
-    <material>Gazebo/FlatBlack</material>
-  </gazebo>
-  <!-- Equivalent to the OpenRAVE manipulator denso_robotiq_85_gripper -->
-  <!-- <link name="denso_robotiq_85_gripper" /> -->
-  <!-- <joint name="manipulator_dummy_joint" type="fixed"> -->
-  <!--   <origin xyz="0 0 0.1441" rpy="0 0 0" /> -->
-  <!--   <parent link="robotiq_coupler"/> -->
-  <!--   <child link="denso_robotiq_85_gripper"/> -->
-  <!-- </joint> -->
-  <!-- Attach the robotiq 85 gripper -->
-  <xacro:robotiq_handE parent="robotiq_coupler" >
-    <origin xyz="0 0 0.088" rpy="${pi*2} ${-4*pi/2} ${pi/2}"/>
-  </xacro:robotiq_handE>
-  <!-- Gazebo FT sensor plugin -->
-  <gazebo reference="wrist_3_joint">
-    <provideFeedback>true</provideFeedback>
-  </gazebo>
-  <link name="end_link"/>
-  <joint name="end_end_joint" type="fixed">
+  <joint name="pedestal_joint" type="fixed">
+    <origin xyz="0.0 0.0 0.25"/>
+    <parent link="pedestal_link"/>
+    <child link="base_link"/>
+  </joint>
+  <joint name="camera_joint" type="fixed">
+    <origin xyz="0.3 0.0 2.0" rpy="0.0 ${pi/2} ${pi/2}"/>
+    <parent link="world"/>
+    <child link="camera_link"/>
+  </joint>
+<link name="camera_link">
+  <visual>
     <origin xyz="0.0 0.0 0.0" rpy="0.0 0.0 0.0"/>
-    <parent link="body_link"/>
-    <child link="end_link"/>
-    <axis xyz="0.0 0.0 0.0"/>
-  </joint>
-  <!--gazebo>
-    <plugin name="ft_sensor_plugin" filename="libgazebo_ros_ft_sensor.so">
-      <updateRate>250.0</updateRate>
-      <topicName>ft_sensor/raw</topicName>
-      <gaussianNoise>0.0</gaussianNoise>
-      <jointName>wrist_3_joint</jointName>
-    </plugin>
-  </gazebo-->
-  <!-- Gazebo grasping plugin -->
-  <!--gazebo>
-    <gripper name="gazebo_gripper">
-      <grasp_check>
-        <attach_steps>2</attach_steps>
-        <detach_steps>2</detach_steps>
-        <min_contact_count>3</min_contact_count>
-      </grasp_check>
-      <gripper_link>robotiq_85_left_finger_tip_link</gripper_link>
-      <gripper_link>robotiq_85_right_finger_tip_link</gripper_link>
-      <palm_link>robotiq_85_base_link</palm_link>
-    </gripper>
-  </gazebo-->
+    <geometry>
+      <box size="0.1 0.1 0.1"/>
+    </geometry>
+    <material name="Cyan">
+      <color rgba="0.0 1.0 0.0 1.0"/>
+    </material>
+  </visual>
+  <collision>
+    <origin xyz="0.0 0.0 0.0" rpy="0.0 0.0 0.0"/>
+    <geometry>
+      <box size="0.1 0.1 0.1"/>
+    </geometry>
+  </collision>
+  <inertial>
+    <origin xyz="0.0 0.0 0.0" rpy="0.0 0.0 0.0"/>
+    <mass value="0.5"/>
+    <inertia ixx="0.01" ixy="0.0" ixz="0.0" iyy="0.01" iyz="0.0" izz="0.01" />
+  </inertial>
+</link>
+<gazebo reference="pedestal_link">
+  <material>Gazebo/Green</material>
+</gazebo>
+<gazebo reference="camera_link">
+  <material>Gazebo/Gray</material>
+  <sensor type="camera" name="camera1">
+      <update_rate>30.0</update_rate>
+      <camera name="head">
+          <horizontal_fov>1.3962634</horizontal_fov>
+          <image>
+          <width>640</width>
+          <height>360</height>
+          <format>R8G8B8</format>
+          </image>
+          <clip>
+          <near>0.02</near>
+          <far>300</far>
+          </clip>
+          <noise>
+          <type>gaussian</type>
+          <mean>0.0</mean>
+          <stddev>0.007</stddev>
+          </noise>
+      </camera>
+      <plugin name="camera_controller" filename="libgazebo_ros_camera.so">
+          <alwaysOn>true</alwaysOn>
+          <updateRate>0.0</updateRate>
+          <cameraName>camera</cameraName>
+          <imageTopicName>image_raw</imageTopicName>
+          <cameraInfoTopicName>camera_info</cameraInfoTopicName>
+          <frameName>camera_link</frameName>
+          <hackBaseline>0.07</hackBaseline>
+          <distortionK1>0.0</distortionK1>
+          <distortionK2>0.0</distortionK2>
+          <distortionK3>0.0</distortionK3>
+          <distortionT1>0.0</distortionT1>
+          <distortionT2>0.0</distortionT2>
+      </plugin>
+  </sensor>
+</gazebo>
 </robot>

File: pick_and_place/urdf/ur3_camera_v2.urdf.xacro (robot description, xacro)
@@ -19,5 +19,5 @@
     kinematics_file="${load_yaml('$(arg kinematics_config)')}"
   />
-  <link name="world_link"/>
+  <link name="world"/>
   <joint name="ur_base_joint" type="fixed">
     <origin xyz="0.0 0.0 0.25" rpy="0.0 0.0 0.0"/>
@@ -33,14 +33,14 @@
     <origin xyz="0.1 0.1 0.4"/>
   </xacro:red_box>
-  <xacro:camera parent="world_link">
+  <xacro:camera parent="world">
     <origin xyz="0.2 0.0 2.0" rpy="0.0 ${pi/2} ${pi/2}"/>
   </xacro:camera>
-  <xacro:pedestal parent="world_link">
+  <xacro:pedestal parent="world">
     <origin xyz="0.0 0.0 0.25"/>
   </xacro:pedestal>
-  <xacro:desk parent="world_link">
+  <xacro:desk parent="world">
     <origin xyz="0.3 0.0 0.0"/>
   </xacro:desk>
-  <xacro:bin parent="world_link">
+  <xacro:bin parent="world">
     <origin xyz="0.0 0.6 0.0"/>
   </xacro:bin>
