Commit message: main

File: pick_and_place/urdf/redbox_v2.urdf.xacro (robot description, xacro)
@@ -4,7 +4,7 @@
     <color rgba="1.0 0.0 0.0 1.0"/>
   </material>
-    <link name="world"/>
+    <link name="world_link"/>
     <joint name="red_box_joint" type="fixed">
-      <parent link="world"/>
+      <parent link="world_link"/>
       <child link="red_box"/>
     </joint>
