Commit message: add

File: arm_and_gripper/arm_and_gripper/urdf/hande.urdf.xacro (robot description, xacro)
@@ -15,5 +15,5 @@
         <link name="body_link">
             <inertial>
-                <origin xyz="0.0 0.0 0.0" />
+                <origin xyz="0.2 0.0 0.0" />
                 <mass value="0.63387"/>
                 <inertia ixx = "0.000002" ixy = "0.000000" ixz = "0.000000"
@@ -37,11 +37,31 @@
             <material>Gazebo/Black</material>
         </gazebo>
+        <!-- <joint name="finger1_joint" type="fixed">
+            <parent link="body_link"/>
+            <child link="finger_11_link"/>
+            <origin xyz="0.0 0.0 0.0" rpy="${-pi/2} ${2*pi/2} 0.0"/>
+            <<axis xyz="0 0 -1"/>
+            <limit effort="130" lower="0" upper="0.025" velocity="0.15"/>
+        </joint> -->
         <joint name="finger1_joint" type="prismatic">
             <parent link="body_link"/>
             <child link="finger_11_link"/>
-            <origin rpy="${-pi/2} ${2*pi/2} 0.0" xyz="0.0 0.0 0.0"/>
+            <origin xyz="0.0 0.0 0.0" rpy="${-pi/2} ${2*pi/2} 0.0"/>
             <axis xyz="0 0 -1"/>
             <limit effort="130" lower="0" upper="0.025" velocity="0.15"/>
         </joint>
+        <!-- <joint name="finger1_joint" type="revolute">
+            <parent link="body_link"/>
+            <child link="finger_11_link"/>
+            <origin xyz="0.0 0.0 0.0" rpy="${-pi/2} ${2*pi/2} 0.0"/>
+            <axis xyz="0 0 -1"/>
+            <limit effort="130" lower="0" upper="0.025" velocity="0.15"/>
+            <limit lower="0" upper="0.7" velocity="2.0" effort="1000" />
+                <limit lower="0" upper="0.7" velocity="2.0" effort="1000" />
+            <xacro:if value="true">
+            <safety_controller soft_lower_limit="${-2.0 * pi}" soft_upper_limit="${2.0 * pi}" k_position="${pi}" k_velocity="0.0"/>
+            </xacro:if>
+            <dynamics damping="0.0" friction="0.0"/>
+        </joint> -->
         <link name="finger_11_link">
             <inertial>
@@ -57,8 +77,8 @@
                 </geometry>
                 <material name="gray" />
-                <!--origin rpy="${pi/2} ${-pi/2} ${pi}" xyz="0.086 0 0"/-->
+                <!-- <origin rpy="${pi/2} ${-pi/2} ${pi}" xyz="0.086 0 0"/> -->
             </visual>
             <collision>
-                <!--origin rpy="${pi/2} ${-pi/2} ${pi}" xyz="0.086 0 0"/-->
+                <!-- <origin rpy="${pi/2} ${-pi/2} ${pi}" xyz="0.086 0 0"/> -->
                 <geometry>
                     <mesh filename="package://arm_and_gripper/meshes/finger_11.dae"/>
@@ -72,12 +92,9 @@
             <mu2 value="0.8"/>
         </gazebo>
-        <!-- <xacro:sensor_d435 parent="body_link">
-            <origin xyz="0.03 0.0 0.0" rpy="${-pi} ${-pi/2} 0.0"/>
-        </xacro:sensor_d435> -->
-        <!-- <joint name="camera_joint" type="fixed">
+        <!--joint name="finger2_joint" type="fixed">
             <parent link="body_link"/>
-            <child link="sensor_d435_link"/>
-            <origin xyz="0.0356 0.0 -0.008" rpy="0.0 ${-pi/2} ${pi/2}"/>
-        </joint> -->
+            <child link="finger_22_link"/>
+            <origin rpy="${-pi/2} ${2*pi/2} 0.0" xyz="0.0 0.02 0.0"/>
+        </joint-->
         <joint name="finger2_joint" type="prismatic">
             <parent link="body_link"/>
@@ -88,4 +105,12 @@
             <mimic joint="finger1_joint" multiplier="1" offset="0"/>
         </joint>
+         <!-- <joint name="finger2_joint" type="fixed">
+            <parent link="body_link"/>
+            <child link="finger_22_link"/>
+            <origin rpy="${-pi/2} ${2*pi/2} 0.0" xyz="0.0 0.0 0.0"/>
+            <axis xyz="0 0 1"/>
+            <limit effort="130" lower="0" upper="0.025" velocity="0.15"/>
+            <mimic joint="finger1_joint" multiplier="1" offset="0"/>
+        </joint> -->
         <link name="finger_22_link">
             <inertial>

File: arm_and_gripper/arm_and_gripper/urdf/ur3e.urdf.xacro (robot description, xacro)
@@ -296,7 +296,8 @@
       </visual>
       <collision>
-        <origin xyz="0 0 -0.0921" rpy="${pi/2} 0 0"/>
-        <geometry>
-          <mesh filename="package://arm_and_gripper/meshes/ur3e/visual/wrist3.dae"/>
+        <origin xyz="0.0 0.0 -0.023" rpy="0.0 0 0"/>
+        <geometry>
+          <!-- <mesh filename="package://arm_and_gripper/meshes/ur3e/visual/wrist3.dae"/> -->
+          <cylinder radius="0.031" length="0.032"/>
         </geometry>
       </collision>

File: realsense2_description/urdf/_d435.urdf.xacro (robot description, xacro)
@@ -48,5 +48,5 @@
         <geometry>
           <!-- <box size="${d435_cam_width} ${d435_cam_height} ${d435_cam_depth}"/> -->
-          <mesh filename="package://realsense2_description/meshes/d435.dae" />
+          <mesh filename="package://realsense2_description/meshes/d435e.dae" />
         </geometry>
         <material name="${name}_aluminum"/>

Commit message: add

File: arm_and_gripper/arm_and_gripper/urdf/hande.urdf.xacro (robot description, xacro)
@@ -17,7 +17,7 @@
                 <origin xyz="0.2 0.0 0.0" />
                 <mass value="0.63387"/>
-                <inertia ixx = "0.000002" ixy = "0.000000" ixz = "0.000000"
-                    iyx = "0.000000" iyy = "0.000005" iyz = "0.000000"
-                    izx = "0.000000" izy = "0.000000" izz = "0.000006" />
+                <inertia ixx = "0.02" ixy = "0.000000" ixz = "0.000000"
+                    iyx = "0.000000" iyy = "0.05" iyz = "0.000000"
+                    izx = "0.000000" izy = "0.000000" izz = "0.06" />
             </inertial>
             <visual>
@@ -68,7 +68,7 @@
                 <origin xyz="0.0 0.0 0.0" />
                 <mass value="0.03804"/>
-                <inertia ixx = "0.000002" ixy = "0.000000" ixz = "0.000000"
-                        iyx = "0.000000" iyy = "0.000005" iyz = "0.000000"
-                        izx = "0.000000" izy = "0.000000" izz = "0.000006" />
+                <inertia ixx = "0.02" ixy = "0.000000" ixz = "0.000000"
+                        iyx = "0.000000" iyy = "0.05" iyz = "0.000000"
+                        izx = "0.000000" izy = "0.000000" izz = "0.06" />
             </inertial>
             <visual>
@@ -118,7 +118,7 @@
                 <!--origin rpy="0 0 0" xyz="-0.02262 0.00759 0.00738"/-->
                 <mass value="0.03804"/>
-                <inertia ixx = "0.000002" ixy = "0.000000" ixz = "0.000000"
-                        iyx = "0.000000" iyy = "0.000005" iyz = "0.000000"
-                        izx = "0.000000" izy = "0.000000" izz = "0.000006" />
+                <inertia ixx = "0.02" ixy = "0.000000" ixz = "0.000000"
+                        iyx = "0.000000" iyy = "0.05" iyz = "0.000000"
+                        izx = "0.000000" izy = "0.000000" izz = "0.06" />
             </inertial>
             <visual>

File: arm_and_gripper/arm_and_gripper/urdf/ur3e.urdf.xacro (robot description, xacro)
@@ -296,8 +296,9 @@
       </visual>
       <collision>
-        <origin xyz="0.0 0.0 -0.023" rpy="0.0 0 0"/>
-        <geometry>
-          <!-- <mesh filename="package://arm_and_gripper/meshes/ur3e/visual/wrist3.dae"/> -->
-          <cylinder radius="0.031" length="0.032"/>
+        <origin xyz="0 0 -0.0921" rpy="${pi/2} 0 0"/>
+        <!-- <origin xyz="0.0 0.0 -0.023" rpy="0.0 0 0"/> -->
+        <geometry>
+          <mesh filename="package://arm_and_gripper/meshes/ur3e/visual/wrist3.dae"/>
+          <!-- <cylinder radius="0.031" length="0.032"/> -->
         </geometry>
       </collision>

File: arm_and_gripper/arm_and_gripper/urdf/ur3e_realsense.urdf.xacro (robot description, xacro)
@@ -41,5 +41,5 @@
     <origin xyz="0 0 0.088" rpy="${pi*2} ${-4*pi/2} ${pi/2}"/>
   </xacro:robotiq_handE>
-  <link name="UR3_camera_mount_upper">
+  <!-- <link name="UR3_camera_mount_upper">
     <visual>
       <geometry>
@@ -77,5 +77,5 @@
     </collision>
     <inertial>
-      <mass value="34.379"/>
+      <mass value="0.034379"/>
       <inertia ixx="7481.438" ixy="0.0" ixz="0.0" iyy="27101.423" iyz="-124.277" izz="29027.607"/>
     </inertial>
@@ -91,5 +91,5 @@
   <xacro:sensor_d435 parent="UR3_camera_mount_upper">
     <origin xyz="0.0 0.04075 0.0075" rpy="0.0 ${-pi/2-pi/10} ${-pi/2}"/>
-  </xacro:sensor_d435>
+  </xacro:sensor_d435> -->
   <!-- Gazebo FT sensor plugin -->
   <gazebo reference="wrist_3_joint">

File: arm_and_gripper/arm_and_gripper/urdf/ur3e_realsense_mount.urdf.xacro (robot description, xacro)
@@ -299,5 +299,5 @@
         <origin xyz="0 0 -0.0921" rpy="${pi/2} 0 0"/>
         <geometry>
-          <mesh filename="package://arm_and_gripper/meshes/ur3e/visual/wrist3.dae"/>
+          <mesh filename="package://arm_and_gripper/meshes/ur3e/collision/wrist3.stl"/>
         </geometry>
       </collision>
@@ -306,5 +306,5 @@
       </xacro:cylinder_inertial>
     </link>
-    <!-- <link name="UR3_camera_mount_upper">
+    <link name="UR3_camera_mount_upper">
     <visual>
       <geometry>
@@ -342,5 +342,5 @@
     </collision>
     <inertial>
-      <mass value="34.379"/>
+      <mass value="0.034379"/>
       <inertia ixx="7481.438" ixy="0.0" ixz="0.0" iyy="27101.423" iyz="-124.277" izz="29027.607"/>
     </inertial>
@@ -356,5 +356,5 @@
   <xacro:sensor_d435 parent="UR3_camera_mount_upper">
     <origin xyz="0.0 0.04075 0.0075" rpy="0.0 ${-pi/2-pi/10} ${-pi/2}"/>
-  </xacro:sensor_d435> -->
+  </xacro:sensor_d435>
     <joint name="${prefix}ee_fixed_joint" type="fixed">
       <parent link="${prefix}wrist_3_link" />
