Commit message: add

File: arm_and_gripper/arm_and_gripper/urdf/ur3e_realsense_mount.urdf.xacro (robot description, xacro)
@@ -309,10 +309,10 @@
     <visual>
       <geometry>
-        <mesh filename="package://arm_and_gripper/meshes/UR3_camera_mount_upper_.dae" />
+        <mesh filename="package://arm_and_gripper/meshes/UR3_camera_mount_lower.dae" />
       </geometry>
     </visual>
     <collision>
       <geometry>
-        <mesh filename="package://arm_and_gripper/meshes/UR3_camera_mount_upper_.dae" />
+        <mesh filename="package://arm_and_gripper/meshes/UR3_camera_mount_lower.dae" />
       </geometry>
     </collision>
@@ -333,10 +333,10 @@
     <visual>
       <geometry>
-        <mesh filename="package://arm_and_gripper/meshes/UR3_camera_mount_lower_.dae" />
+        <mesh filename="package://arm_and_gripper/meshes/UR3_camera_mount_rectangle.dae" />
       </geometry>
     </visual>
     <collision>
       <geometry>
-        <mesh filename="package://arm_and_gripper/meshes/UR3_camera_mount_lower_.dae" />
+        <mesh filename="package://arm_and_gripper/meshes/UR3_camera_mount_rectangle.dae" />
       </geometry>
     </collision>
@@ -354,6 +354,9 @@
     <child link="UR3_camera_mount_lower"/>
   </joint>
-  <xacro:sensor_d435 parent="UR3_camera_mount_upper">
+  <!-- <xacro:sensor_d435 parent="UR3_camera_mount_upper">
     <origin xyz="0.0 0.04075 0.0075" rpy="0.0 ${-pi/2-pi/10} ${-pi/2}"/>
+  </xacro:sensor_d435> -->
+  <xacro:sensor_d435 parent="UR3_camera_mount_lower">
+    <origin xyz="0.0 -0.0421 -0.0075" rpy="0.0 ${pi/2-pi/10} ${-pi/2}"/>
   </xacro:sensor_d435>
     <joint name="${prefix}ee_fixed_joint" type="fixed">

Commit message: add

File: arm_and_gripper/arm_and_gripper/urdf/ur3e_realsense_mount.urdf.xacro (robot description, xacro)
@@ -309,15 +309,15 @@
     <visual>
       <geometry>
-        <mesh filename="package://arm_and_gripper/meshes/UR3_camera_mount_lower.dae" />
+        <mesh filename="package://arm_and_gripper/meshes/UR3_camera_mount_lower_.dae" />
       </geometry>
     </visual>
     <collision>
       <geometry>
-        <mesh filename="package://arm_and_gripper/meshes/UR3_camera_mount_lower.dae" />
+        <mesh filename="package://arm_and_gripper/meshes/UR3_camera_mount_lower_.dae" />
       </geometry>
     </collision>
     <inertial>
       <mass value="0.040837"/>
-      <inertia ixx="9901" ixy="0.023" ixz="-0.009" iyy="28968.111" iyz="1072.256" izz="33057.788"/>
+      <inertia ixx="9901e-09" ixy="0.023e-09" ixz="-0.009e-09" iyy="28968.111e-09" iyz="1072.256e-09" izz="33057.788e-09"/>
     </inertial>
   </link>
@@ -333,15 +333,15 @@
     <visual>
       <geometry>
-        <mesh filename="package://arm_and_gripper/meshes/UR3_camera_mount_rectangle.dae" />
+        <mesh filename="package://arm_and_gripper/meshes/UR3_camera_mount_rectangle_.dae" />
       </geometry>
     </visual>
     <collision>
       <geometry>
-        <mesh filename="package://arm_and_gripper/meshes/UR3_camera_mount_rectangle.dae" />
+        <mesh filename="package://arm_and_gripper/meshes/UR3_camera_mount_rectangle_.dae" />
       </geometry>
     </collision>
     <inertial>
       <mass value="0.034379"/>
-      <inertia ixx="7481.438" ixy="0.0" ixz="0.0" iyy="27101.423" iyz="-124.277" izz="29027.607"/>
+      <inertia ixx="7481.438e-09" ixy="0.0" ixz="0.0" iyy="27101.423e-09" iyz="-124.277e-09" izz="29027.607e-09"/>
     </inertial>
   </link>
