Commit message: add

File: arm_and_gripper/arm_and_gripper/urdf/robotiq_85_gripper/robotiq_85_gripper.transmission.xacro (robot description, xacro)
@@ -16,17 +16,17 @@
     <!-- Mimic joints -->
     <gazebo>
-      <plugin filename="libgazebo_mimic_joint_plugin.so" name="${prefix}mimic_robotiq_85_1">
+      <plugin filename="libroboticsgroup_upatras_gazebo_mimic_joint_plugin.so" name="${prefix}mimic_robotiq_85_1">
         <joint>${prefix}robotiq_85_left_knuckle_joint</joint>
         <mimicJoint>${prefix}robotiq_85_right_knuckle_joint</mimicJoint>
       </plugin>
-      <plugin filename="libgazebo_mimic_joint_plugin.so" name="${prefix}mimic_robotiq_85_2">
+      <plugin filename="libroboticsgroup_upatras_gazebo_mimic_joint_plugin.so" name="${prefix}mimic_robotiq_85_2">
         <joint>${prefix}robotiq_85_left_knuckle_joint</joint>
         <mimicJoint>${prefix}robotiq_85_left_inner_knuckle_joint</mimicJoint>
       </plugin>
-      <plugin filename="libgazebo_mimic_joint_plugin.so" name="${prefix}mimic_robotiq_85_3">
+      <plugin filename="libroboticsgroup_upatras_gazebo_mimic_joint_plugin.so" name="${prefix}mimic_robotiq_85_3">
         <joint>${prefix}robotiq_85_left_knuckle_joint</joint>
         <mimicJoint>${prefix}robotiq_85_right_inner_knuckle_joint</mimicJoint>
       </plugin>
-      <plugin filename="libgazebo_mimic_joint_plugin.so" name="${prefix}mimic_robotiq_85_4">
+      <plugin filename="libroboticsgroup_upatras_gazebo_mimic_joint_plugin.so" name="${prefix}mimic_robotiq_85_4">
         <joint>${prefix}robotiq_85_left_knuckle_joint</joint>
         <mimicJoint>${prefix}robotiq_85_left_finger_tip_joint</mimicJoint>
@@ -34,5 +34,5 @@
         <offset>0.0</offset>
       </plugin>
-      <plugin filename="libgazebo_mimic_joint_plugin.so" name="${prefix}mimic_robotiq_85_5">
+      <plugin filename="libroboticsgroup_upatras_gazebo_mimic_joint_plugin.so" name="${prefix}mimic_robotiq_85_5">
         <joint>${prefix}robotiq_85_left_knuckle_joint</joint>
         <mimicJoint>${prefix}robotiq_85_right_finger_tip_joint</mimicJoint>

File: arm_and_gripper/arm_and_gripper/urdf/robotiq_85_gripper/robotiq_85_gripper.urdf.xacro (robot description, xacro)
@@ -35,4 +35,5 @@
     </joint>
     <joint name="${prefix}robotiq_85_right_knuckle_joint" type="continuous">
+    <!-- <joint name="${prefix}robotiq_85_right_knuckle_joint" type="revolute"> -->
       <parent link="${prefix}robotiq_85_base_link"/>
       <child link="${prefix}robotiq_85_right_knuckle_link"/>
@@ -129,4 +130,5 @@
     </link>
     <joint name="${prefix}robotiq_85_left_inner_knuckle_joint" type="continuous">
+    <!-- <joint name="${prefix}robotiq_85_left_inner_knuckle_joint" type="revolute"> -->
       <parent link="${prefix}robotiq_85_base_link"/>
       <child link="${prefix}robotiq_85_left_inner_knuckle_link"/>
@@ -137,4 +139,5 @@
     </joint>
     <joint name="${prefix}robotiq_85_right_inner_knuckle_joint" type="continuous">
+    <!-- <joint name="${prefix}robotiq_85_right_inner_knuckle_joint" type="revolute"> -->
       <parent link="${prefix}robotiq_85_base_link"/>
       <child link="${prefix}robotiq_85_right_inner_knuckle_link"/>
@@ -183,4 +186,5 @@
     </link>
     <joint name="${prefix}robotiq_85_left_finger_tip_joint" type="continuous">
+    <!-- <joint name="${prefix}robotiq_85_left_finger_tip_joint" type="revolute"> -->
       <parent link="${prefix}robotiq_85_left_inner_knuckle_link"/>
       <child link="${prefix}robotiq_85_left_finger_tip_link"/>
@@ -191,4 +195,5 @@
     </joint>
     <joint name="${prefix}robotiq_85_right_finger_tip_joint" type="continuous">
+    <!-- <joint name="${prefix}robotiq_85_right_finger_tip_joint" type="revolute"> -->
       <parent link="${prefix}robotiq_85_right_inner_knuckle_link"/>
       <child link="${prefix}robotiq_85_right_finger_tip_link"/>

File: arm_and_gripper/arm_and_gripper/urdf/ur3e_85_realsense/ur3e_85_realsense.urdf.xacro (robot description, xacro)
@@ -28,5 +28,5 @@
   </link>
   <joint name="robotiq_coupler_joint" type="fixed">
-    <!--origin xyz="0 0 0.004" rpy="0 0 ${pi}" /-->
+    <origin xyz="0 0 0.004" rpy="0 0 ${pi/2}" />
     <parent link="tool0"/>
     <child link="robotiq_coupler"/>
@@ -39,5 +39,5 @@
   <!-- Attach the robotiq 85 gripper -->
   <xacro:robotiq_85_gripper prefix="" parent="robotiq_coupler" >
-    <origin xyz="0 0 0.004" rpy="${pi/2} ${-pi/2} ${pi}"/>
+    <origin xyz="0 0 0.005" rpy="0 ${-pi/2} ${pi}"/>
   </xacro:robotiq_85_gripper>
   <!-- Gazebo FT sensor plugin -->
