Commit message: add

File: arm_and_gripper/arm_and_gripper/urdf/robotiq_85_gripper/robotiq_85_gripper.urdf.xacro (robot description, xacro)
@@ -34,6 +34,6 @@
       <limit lower="0.0" upper="0.80285" velocity="0.5" effort="1000"/>
     </joint>
-    <joint name="${prefix}robotiq_85_right_knuckle_joint" type="continuous">
-    <!-- <joint name="${prefix}robotiq_85_right_knuckle_joint" type="revolute"> -->
+    <!-- <joint name="${prefix}robotiq_85_right_knuckle_joint" type="continuous"> -->
+    <joint name="${prefix}robotiq_85_right_knuckle_joint" type="revolute">
       <parent link="${prefix}robotiq_85_base_link"/>
       <child link="${prefix}robotiq_85_right_knuckle_link"/>
@@ -129,6 +129,6 @@
       </inertial>
     </link>
-    <joint name="${prefix}robotiq_85_left_inner_knuckle_joint" type="continuous">
-    <!-- <joint name="${prefix}robotiq_85_left_inner_knuckle_joint" type="revolute"> -->
+    <!-- <joint name="${prefix}robotiq_85_left_inner_knuckle_joint" type="continuous"> -->
+    <joint name="${prefix}robotiq_85_left_inner_knuckle_joint" type="revolute">
       <parent link="${prefix}robotiq_85_base_link"/>
       <child link="${prefix}robotiq_85_left_inner_knuckle_link"/>
@@ -138,6 +138,6 @@
       <mimic joint="${prefix}robotiq_85_left_knuckle_joint" offset="0"/>
     </joint>
-    <joint name="${prefix}robotiq_85_right_inner_knuckle_joint" type="continuous">
-    <!-- <joint name="${prefix}robotiq_85_right_inner_knuckle_joint" type="revolute"> -->
+    <!-- <joint name="${prefix}robotiq_85_right_inner_knuckle_joint" type="continuous"> -->
+    <joint name="${prefix}robotiq_85_right_inner_knuckle_joint" type="revolute">
       <parent link="${prefix}robotiq_85_base_link"/>
       <child link="${prefix}robotiq_85_right_inner_knuckle_link"/>
@@ -185,6 +185,6 @@
       </inertial>
     </link>
-    <joint name="${prefix}robotiq_85_left_finger_tip_joint" type="continuous">
-    <!-- <joint name="${prefix}robotiq_85_left_finger_tip_joint" type="revolute"> -->
+    <!-- <joint name="${prefix}robotiq_85_left_finger_tip_joint" type="continuous"> -->
+    <joint name="${prefix}robotiq_85_left_finger_tip_joint" type="revolute">
       <parent link="${prefix}robotiq_85_left_inner_knuckle_link"/>
       <child link="${prefix}robotiq_85_left_finger_tip_link"/>
@@ -194,6 +194,6 @@
       <mimic joint="${prefix}robotiq_85_left_knuckle_joint" multiplier="-1"/>
     </joint>
-    <joint name="${prefix}robotiq_85_right_finger_tip_joint" type="continuous">
-    <!-- <joint name="${prefix}robotiq_85_right_finger_tip_joint" type="revolute"> -->
+    <!-- <joint name="${prefix}robotiq_85_right_finger_tip_joint" type="continuous"> -->
+    <joint name="${prefix}robotiq_85_right_finger_tip_joint" type="revolute">
       <parent link="${prefix}robotiq_85_right_inner_knuckle_link"/>
       <child link="${prefix}robotiq_85_right_finger_tip_link"/>
