Commit message: add

File: arm_and_gripper/arm_and_gripper/urdf/ur3e_85_realsense/ur3e_85_realsense.urdf.xacro (robot description, xacro)
@@ -39,5 +39,5 @@
   <!-- Attach the robotiq 85 gripper -->
   <xacro:robotiq_85_gripper prefix="" parent="robotiq_coupler" >
-    <origin xyz="0 0 0.005" rpy="0 ${-pi/2} ${pi}"/>
+    <origin xyz="0 0 0.004" rpy="0 ${-pi/2} ${pi}"/>
   </xacro:robotiq_85_gripper>
   <!-- Gazebo FT sensor plugin -->
